Commit message: fix(urdf): base_link as root, base_footprint as ground-projection leaf
The joint was base_footprint->base_link while both EKFs use base_link_frame=base_link and the ESP32 wheel odom reports child_frame_id=base_link, giving base_link two parents (odom + base_footprint) and orphaning base_footprint from map (RViz: 'No transform from base_footprint to map'). Flip to base_link->base_footprint (z=-base_height) so the tree is map->odom->base_link->{base_footprint,gnss_link,wheels}.

File: src/outdoor_patrol_bringup/urdf/outdoor_patrol.urdf.xacro (robot description, xacro)
@@ -5,7 +5,8 @@
     config/chassis.yaml (single source of truth) — adjust dimensions and
     sensor placements THERE, not in this file.
-    Frames follow REP-105: base_footprint (ground) -> base_link (chassis),
-    with module frames (gnss_link, …) hung off base_link from the yaml
-    `modules:` section.
+    Frames follow REP-105: base_link (chassis) is the estimated body frame
+    (the EKFs publish odom -> base_link, matching the wheel-odom child frame),
+    with base_footprint as its ground projection hung below it, and module
+    frames (gnss_link, …) hung off base_link from the yaml `modules:` section.
     Wheel joints are FIXED until a joint-state source exists (M1+ switches
     them to 'continuous' when odometry / ros2_control feeds joint_states).
@@ -35,8 +36,8 @@
     </visual>
   </link>
-  <joint name="base_footprint_to_base_link" type="fixed">
-    <parent link="base_footprint"/>
-    <child  link="base_link"/>
-    <origin xyz="0 0 ${base_height}" rpy="0 0 0"/>
+  <joint name="base_link_to_base_footprint" type="fixed">
+    <parent link="base_link"/>
+    <child  link="base_footprint"/>
+    <origin xyz="0 0 ${-base_height}" rpy="0 0 0"/>
   </joint>
   <!-- ── Wheels ───────────────────────────────────────────────────── -->

Commit message: fix(bringup): center body visual box on wheel axle (offset 0.22 m forward)
The cosmetic chassis box was drawn centered on base_link, but the body actually sits 0.22 m forward of the wheel axle. Add body_offset_x and shift the base_link visual origin; also correct the box footprint to 0.64x0.44. RViz-only, no effect on TF/collision/EKF.

File: src/outdoor_patrol_bringup/urdf/outdoor_patrol.urdf.xacro (robot description, xacro)
@@ -23,9 +23,10 @@
   <xacro:property name="body_width"       value="${ch['body_width']}"/>
   <xacro:property name="body_height"      value="${ch['body_height']}"/>
+  <xacro:property name="body_offset_x"    value="${ch['body_offset_x']}"/>
   <!-- base_footprint sits on the ground directly below base_link. -->
   <link name="base_footprint"/>
   <link name="base_link">
     <visual>
-      <origin xyz="0 0 0" rpy="0 0 0"/>
+      <origin xyz="${body_offset_x} 0 0" rpy="0 0 0"/>
       <geometry>
         <box size="${body_length} ${body_width} ${body_height}"/>

Commit message: feat(bringup): add imu_link frame + map IMU device for M2 bring-up
Add the Inertial Labs KERNEL IMU to the robot description and expose it to
the robot container for standalone bring-up (M2; no EKF fusion yet).

- chassis.yaml: imu_link module at xyz "0.281 0 0.17", rpy "0 -1.5708
  3.14159" (sensor X->up, Y->right, Z->forward); verified to map sensor axes
  to base_link. Confirm physically with the level + yaw-sign test.
- outdoor_patrol.urdf.xacro: module_frame call so robot_state_publisher owns
  base_link->imu_link.
- deploy/docker-compose.yaml: map the FTDI FT230X IMU by-id device (IMU_DEV
  override).

File: src/outdoor_patrol_bringup/urdf/outdoor_patrol.urdf.xacro (robot description, xacro)
@@ -80,3 +80,6 @@
   <xacro:module_frame name="gnss_link" parent="${gnss['parent']}"
                       xyz="${gnss['xyz']}" rpy="${gnss['rpy']}"/>
+  <xacro:property name="imu" value="${modules['imu_link']}"/>
+  <xacro:module_frame name="imu_link" parent="${imu['parent']}"
+                      xyz="${imu['xyz']}" rpy="${imu['rpy']}"/>
 </robot>

Commit message: M3: 2D RPLIDAR C1 obstacle avoidance + scan_safety brake (ADR-013)
- sllidar_ros2 submodule (Slamtec C1 driver) + ros2.repos entry.

- New outdoor_patrol_safety pkg: scan_safety forward brake (gates /cmd_vel_raw->/cmd_vel; reverse+rotation pass; fail-safe on stale scan).

- chassis.yaml/urdf: lidar_link 0.512 0 0.05 rpy 0; sensor is LEFT-handed so the mirror is fixed in scan data via driver inverted:=true (empirically confirmed).

- gnss_localization.launch: RPLIDAR (inverted, frame_id lidar_link) + scan_safety, delayed via TimerAction, use_lidar toggle. compose: LIDAR_DEV by-id map + lidar_dev arg.

- Bump robot-research (ADR-013 + M3/M4/M7 plan).

File: src/outdoor_patrol_bringup/urdf/outdoor_patrol.urdf.xacro (robot description, xacro)
@@ -83,3 +83,6 @@
   <xacro:module_frame name="imu_link" parent="${imu['parent']}"
                       xyz="${imu['xyz']}" rpy="${imu['rpy']}"/>
+  <xacro:property name="lidar" value="${modules['lidar_link']}"/>
+  <xacro:module_frame name="lidar_link" parent="${lidar['parent']}"
+                      xyz="${lidar['xyz']}" rpy="${lidar['rpy']}"/>
 </robot>
