Commit message: Add Gazebo Harmonic simulation (outdoor_patrol_sim)
Replaces the whole physical stack -- ESP32-S3 chassis controller, UM982
GNSS, UMKA IMU, RPLIDAR C1 -- with a gz-sim model that publishes on the
SAME ROS topic names the real drivers use, so outdoor_patrol_loc runs
against it with no remaps. Headless by default (works over SSH and in the
dev container); gui:=true for the Gazebo GUI.

The robot description stays shared: outdoor_patrol.urdf.xacro gains a
`sim` xacro arg that adds <collision>/<inertial> blocks and makes the
wheel joints continuous. With sim:=false the rendered URDF is unchanged,
so the hardware path is untouched. Geometry still lives in chassis.yaml,
which gains sim-only mass estimates for the inertia tensors.

Two shim nodes exist because a gz message is missing a field the
localization stack treats as load-bearing:

  * odom_sim  -- the DiffDrive plugin publishes zero odom covariance,
    which robot_localization reads as "infinitely trustworthy"; the EKF
    would ride perfect wheel odometry and ignore GNSS. Stamps the same
    fixed diagonal the firmware sends.
  * gnss_sim  -- adds the covariance gz.msgs.NavSat cannot carry, adds
    the position noise in METRES (gz applies navsat <position_sensing>
    noise in degrees, so a plausible 0.02 throws the fix kilometres off),
    and synthesises /gnss/heading, which ekf_global needs as its only
    absolute-yaw source and the single-antenna gz sensor cannot provide.

Verified headless: settles at exactly the 0.150 m ride height, 10 s at
0.4 m/s covers 4.006 m, /scan at 9.8 Hz reads the geometrically correct
4.19 m to the obstacle at x=5, the fix lands on the world datum within
2 cm, and the global EKF tracks /odom_truth to ~10 cm while driving.

Known differences from the robot are documented in the package README:
no /cmd_vel watchdog, no RTK degradation path, idealised wheel odometry.

Co-authored-by: Copilot <223556219+Copilot@users.noreply.github.com>

File: src/outdoor_patrol_bringup/urdf/outdoor_patrol.urdf.xacro (robot description, xacro)
@@ -11,9 +11,40 @@
     Wheel joints are FIXED until a joint-state source exists (M1+ switches
     them to 'continuous' when odometry / ros2_control feeds joint_states).
+    sim:=true (Gazebo, outdoor_patrol_sim) additionally emits <collision> and
+    <inertial> blocks and makes the wheel joints 'continuous' so the physics
+    engine can drive them. With sim:=false (the default, i.e. the real robot)
+    the output is byte-identical to before this flag existed.
   -->
+  <xacro:arg name="sim" default="false"/>
+  <xacro:property name="sim" value="$(arg sim)"/>
   <!-- ── Config: single source of truth (config/chassis.yaml) ─────── -->
   <xacro:property name="cfg"
       value="${xacro.load_yaml('$(find outdoor_patrol_bringup)/config/chassis.yaml')}"/>
   <xacro:property name="ch" value="${cfg['chassis']}"/>
+  <!-- Masses are only consumed when sim:=true. -->
+  <xacro:property name="body_mass"  value="${ch['body_mass']}"/>
+  <xacro:property name="wheel_mass" value="${ch['wheel_mass']}"/>
+  <!-- Solid-box inertia tensor about its own center. -->
+  <xacro:macro name="box_inertial" params="mass x y z *origin">
+    <inertial>
+      <xacro:insert_block name="origin"/>
+      <mass value="${mass}"/>
+      <inertia ixx="${mass * (y*y + z*z) / 12.0}" ixy="0.0" ixz="0.0"
+               iyy="${mass * (x*x + z*z) / 12.0}" iyz="0.0"
+               izz="${mass * (x*x + y*y) / 12.0}"/>
+    </inertial>
+  </xacro:macro>
+  <!-- Solid-cylinder inertia, spun about Y (wheel axis) after the rpy below. -->
+  <xacro:macro name="wheel_inertial" params="mass radius length">
+    <inertial>
+      <origin xyz="0 0 0" rpy="${pi/2} 0 0"/>
+      <mass value="${mass}"/>
+      <inertia ixx="${mass * (3*radius*radius + length*length) / 12.0}"
+               ixy="0.0" ixz="0.0"
+               iyy="${mass * (3*radius*radius + length*length) / 12.0}"
+               iyz="0.0"
+               izz="${mass * radius * radius / 2.0}"/>
+    </inertial>
+  </xacro:macro>
   <xacro:property name="wheel_radius"     value="${ch['wheel_radius']}"/>
   <xacro:property name="wheel_separation" value="${ch['wheel_separation']}"/>
@@ -36,4 +67,16 @@
       </material>
     </visual>
+    <xacro:if value="${sim}">
+      <collision>
+        <origin xyz="${body_offset_x} 0 0" rpy="0 0 0"/>
+        <geometry>
+          <box size="${body_length} ${body_width} ${body_height}"/>
+        </geometry>
+      </collision>
+      <xacro:box_inertial mass="${body_mass}" x="${body_length}"
+                          y="${body_width}" z="${body_height}">
+        <origin xyz="${body_offset_x} 0 0" rpy="0 0 0"/>
+      </xacro:box_inertial>
+    </xacro:if>
   </link>
   <joint name="base_link_to_base_footprint" type="fixed">
@@ -54,6 +97,17 @@
         </material>
       </visual>
+      <xacro:if value="${sim}">
+        <collision>
+          <origin xyz="0 0 0" rpy="${pi/2} 0 0"/>
+          <geometry>
+            <cylinder radius="${wheel_radius}" length="${wheel_width}"/>
+          </geometry>
+        </collision>
+        <xacro:wheel_inertial mass="${wheel_mass}" radius="${wheel_radius}"
+                              length="${wheel_width}"/>
+      </xacro:if>
     </link>
-    <joint name="${prefix}_wheel_joint" type="fixed">
+    <joint name="${prefix}_wheel_joint"
+           type="${'continuous' if sim else 'fixed'}">
       <parent link="base_link"/>
       <child  link="${prefix}_wheel_link"/>
